File: kicad_data_Title72/Title72.kicad_sch (KiCad schematic)
At the start: 174 parts, among them SW1 SW_PUSH, SW10 SW_PUSH, SW11 SW_PUSH, SW12 SW_PUSH, SW13 SW_PUSH, SW14 SW_PUSH, SW15 SW_PUSH, SW18 SW_SPDT, SW19 SW_PUSH, SW2 SW_PUSH, SW20 SW_PUSH, SW21 SW_PUSH, SW22 SW_PUSH, SW23 SW_PUSH, SW24 SW_PUSH, SW25 SW_PUSH, SW26 SW_PUSH, SW27 SW_PUSH, SW28 SW_PUSH, SW29 SW_PUSH, SW3 SW_PUSH, SW30 SW_PUSH, SW31 SW_PUSH, SW32 SW_PUSH, SW33 SW_PUSH, SW37 SW_PUSH, SW38 SW_PUSH, SW39 SW_PUSH, SW4 SW_PUSH, SW40 SW_PUSH, SW41 SW_PUSH, SW42 SW_PUSH, SW43 SW_PUSH, SW44 SW_PUSH, SW45 SW_PUSH, SW46 SW_PUSH, SW47 SW_PUSH, SW48 SW_PUSH, SW49 SW_PUSH, SW5 SW_PUSH, SW50 SW_PUSH, SW55 SW_PUSH, SW56 SW_PUSH, SW57 SW_PUSH, SW58 SW_PUSH, SW59 SW_PUSH, SW6 SW_PUSH, SW60 SW_PUSH, SW61 SW_PUSH, SW62 SW_PUSH, SW63 SW_PUSH, SW64 SW_PUSH, SW65 SW_PUSH, SW66 SW_PUSH, SW67 SW_PUSH, SW68 SW_PUSH, SW7 SW_PUSH, SW73 SW_PUSH, SW74 SW_PUSH, SW75 SW_PUSH, SW76 SW_PUSH, SW77 SW_PUSH, SW78 SW_PUSH, SW79 SW_PUSH, SW8 SW_PUSH, SW80 SW_PUSH, SW81 SW_PUSH, SW82 SW_PUSH, SW83 SW_PUSH, SW84 SW_PUSH, SW85 SW_PUSH, SW86 SW_PUSH, SW87 SW_PUSH, SW88 SW_PUSH, SW89 SW_PUSH, SW9 SW_DIP_x01, SW9 SW_PUSH, U1 xiao-ble

Commit message: update for jis layout
Parts:
- added D16: D, Diode_SMD:D_SOD-123, symbol Device:D
- added SW16: SW_PUSH, kbd_SW:Choc_v2_Hotswap_1u, symbol Switch:SW_Push
Connections:
- net S6: now also D16.1 (K)
- net at D302.1 (K), D402.1 (K), SW10.1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: now also SW16.1
- new net: D16.2 (A), SW16.2
Changed lines of the file:
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@@
 	)
 	(junction
+		(at 153.67 50.8)
+		(diameter 0)
+		(color 0 0 0 0)
+	)
+	(junction
 		(at 137.16 50.8)
 		(diameter 0)
@@
 	)
 	(junction
+		(at 146.05 60.96)
+		(diameter 0)
+		(color 0 0 0 0)
+	)
+	(junction
 		(at 129.54 166.37)
 		(diameter 0)
@@
 	(wire
 		(pts
-			(xy 146.05 44.45) (xy 146.05 78.74)
+			(xy 146.05 44.45) (xy 146.05 60.96)
 		)
 		(stroke
@@
 	(wire
 		(pts
-			(xy 137.16 50.8) (xy 189.23 50.8)
+			(xy 137.16 50.8) (xy 153.67 50.8)
 		)
 		(stroke
@@
 	(wire
 		(pts
+			(xy 153.67 50.8) (xy 189.23 50.8)
+		)
+		(stroke
+			(width 0)
+			(type default)
+		)
+	)
+	(wire
+		(pts
 			(xy 67.31 120.65) (xy 83.82 120.65)
 		)
@@
 	(wire
 		(pts
+			(xy 146.05 60.96) (xy 146.05 78.74)
+		)
+		(stroke
+			(width 0)
+			(type default)
+		)
+	)
+	(wire
+		(pts
 			(xy 267.97 33.02) (xy 267.97 36.83)
 		)
@@
 	(symbol
 		(lib_id "Device:D")
+		(at 149.86 60.96 0)
+		(unit 1)
+		(exclude_from_sim no)
+		(in_bom yes)
+		(on_board yes)
+		(dnp no)
+		(fields_autoplaced yes)
+		(property "Reference" "D16"
+			(at 149.86 54.61 0)
+			(effects
+				(font
+					(size 1.27 1.27)
+				)
+			)
+		)
+		(property "Value" "D"
+			(at 149.86 57.15 0)
+			(effects
+				(font
+					(size 1.27 1.27)
+				)
+			)
+		)
+		(property "Footprint" "Diode_SMD:D_SOD-123"
+			(at 149.86 60.96 0)
+			(effects
+				(font
+					(size 1.27 1.27)
+				)
+				(hide yes)
+			)
+		)
+		(property "Datasheet" "~"
+			(at 149.86 60.96 0)
+			(effects
+				(font
+					(size 1.27 1.27)
+				)
+				(hide yes)
+			)
+		)
+		(property "Description" ""
+			(at 149.86 60.96 0)
+			(effects
+				(font
+					(size 1.27 1.27)
+				)
+				(hide yes)
+			)
+		)
+		(pin "1"
+		)
+		(pin "2"
+		)
+		(instances
+			(project "Title72"
+				(path "/869844b0-69c5-413c-97b4-f2799caa50e2"
+					(reference "D16")
+					(unit 1)
+				)
+			)
+		)
+	)
+	(symbol
+		(lib_id "Device:D")
 		(at 133.35 130.81 0)
 		(unit 1)
@@
 					(unit 1)
 				)
+			)
+		)
+	)
+	(symbol
+		(lib_id "Switch:SW_Push")
+		(at 153.67 55.88 270)
+		(unit 1)
+		(exclude_from_sim no)
+		(in_bom yes)
+		(on_board yes)
+		(dnp no)
+		(fields_autoplaced yes)
+		(property "Reference" "SW16"
+			(at 157.48 54.6099 90)
+			(effects
+				(font
+					(size 1.27 1.27)
+				)
+				(justify left)
+			)
+		)
+		(property "Value" "SW_PUSH"
+			(at 157.48 57.1499 90)
+			(effects
+				(font
+					(size 1.27 1.27)
+				)
+				(justify left)
+			)
+		)
+		(property "Footprint" "kbd_SW:Choc_v2_Hotswap_1u"
+			(at 158.75 55.88 0)
+			(effects
+				(font
+					(size 1.27 1.27)
+				)
+				(hide yes)
+			)
+		)
+		(property "Datasheet" "~"
+			(at 158.75 55.88 0)
+			(effects
+				(font
+					(size 1.27 1.27)
+				)
+				(hide yes)
+			)
+		)
+		(property "Description" ""
+			(at 153.67 55.88 0)
+			(effects
+				(font
+					(size 1.27 1.27)
+				)
+				(hide yes)
+			)
+		)
+		(pin "1"
+		)
+		(pin "2"
+		)
+		(instances
+			(project "Title72"
+				(path "/869844b0-69c5-413c-97b4-f2799caa50e2"
+					(reference "SW16")
+					(unit 1)
+				)
